File: Hardware/SPIFEE/68k_Cpu.kicad_sch (KiCad schematic)
At the start: 53 parts, among them J301 Conn_02x03, U301 DS1086LU+, U302 MC68SEC000FU, U303 74LVC2G07, U304 74LVC3G06, U305 SST39SF040-55

Commit message: Doc update
Parts:
- U305: value SST39SF040-55 -> SST39LF040-55
Changed lines of the file:
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@@
 			)
 		)
-		(property "Value" "SST39SF040-55"
+		(property "Value" "SST39LF040-55"
 			(at 226.9333 35.56 0)
 			(show_name no)
